File: fullSeveNelson/fullSeveNelson.kicad_sch (KiCad schematic)
At the start: 21 parts, among them J1 USB_C_Receptacle_USB2.0, U1 STM32F072CBT6, U2 PRTR5V0U2X

Commit message: fixed footprints
Parts:
- gave numbers to parts that had none: 15
